Commit message: Add files

File: robot/urdf/parameters.xacro (robot description, xacro)
@@ -19,6 +19,6 @@
 <xacro:property name="cameraY" value="0.04"/>
 <xacro:property name="cameraZ" value="0.06"/>
-<xacro:property name="mesh_chassis"  value="/home/andreag/catkin_ws/src/adjic_autonomousnavigation_puzzlebot/adjic_autonomousnavigation_puzzlebot/meshes/chassis.stl" />
-<xacro:property name="mesh_wheel"  value="/home/andreag/catkin_ws/src/adjic_autonomousnavigation_puzzlebot/adjic_autonomousnavigation_puzzlebot/meshes/wheel.stl" />
-<xacro:property name="mesh_camera"  value="/home/andreag/catkin_ws/src/adjic_autonomousnavigation_puzzlebot/adjic_autonomousnavigation_puzzlebot/meshes/camera.stl" />
+<xacro:property name="mesh_chassis"  value="$(find final_challenge)/robot/meshes/chassis.stl" />
+<xacro:property name="mesh_wheel"  value="$(find final_challenge)/robot/meshes/wheel.stl" />
+<xacro:property name="mesh_camera"  value="$(find final_challenge)/robot/meshes/camera.stl" />
 </robot>

File: robot/urdf/parameters_real.xacro (robot description, xacro)
@@ -19,6 +19,6 @@
 <xacro:property name="cameraY" value="0.04"/>
 <xacro:property name="cameraZ" value="0.06"/>
-<xacro:property name="mesh_chassis"  value="$(find adjic_autonomousnavigation_puzzlebot)/meshes/chassis.stl" />
-<xacro:property name="mesh_wheel"  value="$(find adjic_autonomousnavigation_puzzlebot)/meshes/wheel.stl" />
-<xacro:property name="mesh_camera"  value="$(find adjic_autonomousnavigation_puzzlebot)/meshes/camera.stl" />
+<xacro:property name="mesh_chassis"  value="$(find final_challenge)/robot/meshes/chassis.stl" />
+<xacro:property name="mesh_wheel"  value="$(find final_challenge)/robot/meshes/wheel.stl" />
+<xacro:property name="mesh_camera"  value="$(find final_challenge)/robot/meshes/camera.stl" />
 </robot>

File: robot/urdf/puzzlebot_lidar.xacro (robot description, xacro)
@@ -3,8 +3,8 @@
 <robot name="puzzlebot" xmlns:xacro="http://www.ros.org/wiki/xacro">
 <!-- files for gazebo costumization -->
-<xacro:include filename="$(find adjic_autonomousnavigation_puzzlebot)/urdf/materials.xacro" />
-<xacro:include filename="$(find adjic_autonomousnavigation_puzzlebot)/urdf/parameters.xacro" />
-<xacro:include filename="$(find adjic_autonomousnavigation_puzzlebot)/urdf/puzzlebot.gazebo" />
-<xacro:include filename="$(find adjic_autonomousnavigation_puzzlebot)/urdf/macros.xacro" />
+<xacro:include filename="$(find final_challenge)/robot/urdf/materials.xacro" />
+<xacro:include filename="$(find final_challenge)/robot/urdf/parameters.xacro" />
+<xacro:include filename="$(find final_challenge)/robot/urdf/puzzlebot.gazebo" />
+<xacro:include filename="$(find final_challenge)/robot/urdf/macros.xacro" />
 <!-- Dummy link to fiz robot chassis -->
   <link name="base_link">
